Commit message: WIP rtabmap and rviz

File: ros/t_top/urdf/ttop.urdf.xacro (robot description, xacro)
@@ -46,5 +46,5 @@
       <origin xyz="0     0    0" rpy="0 0 0"/>
       <geometry>
-        <mesh filename="package://ttop_sim/models/ttop/meshes/rotating_base_mesh.dae" scale="1.0 1.0 1.0"/>
+        <mesh filename="package://t_top/meshes/rotating_base_mesh.dae" scale="1.0 1.0 1.0"/>
       </geometry>
     </collision>
@@ -53,5 +53,5 @@
       <origin xyz="0     0    0" rpy="0 0 0"/>
       <geometry>
-        <mesh filename="package://ttop_sim/models/ttop/meshes/rotating_base_mesh.dae" scale="1.0 1.0 1.0"/>
+        <mesh filename="package://t_top/meshes/rotating_base_mesh.dae" scale="1.0 1.0 1.0"/>
       </geometry>
     </visual>
@@ -68,5 +68,5 @@
       <origin xyz="0      0      0" rpy="0       0      0"/>
       <geometry>
-        <mesh filename="package://ttop_sim/models/ttop/meshes/stewart_platform_mesh.dae" scale="1.0 1.0 1.0"/>
+        <mesh filename="package://t_top/meshes/stewart_platform_mesh.dae" scale="1.0 1.0 1.0"/>
       </geometry>
     </collision>
@@ -76,5 +76,5 @@
       <origin xyz="0      0      0" rpy="0       0      0"/>
       <geometry>
-        <mesh filename="package://ttop_sim/models/ttop/meshes/stewart_platform_mesh.dae" scale="1.0 1.0 1.0"/>
+        <mesh filename="package://t_top/meshes/stewart_platform_mesh.dae" scale="1.0 1.0 1.0"/>
       </geometry>
     </visual>
