File: PCB/dynamixel_control/dynamixel.kicad_sch (KiCad schematic)
At the start: 19 parts, among them J11 Dynamixel TTL, J12 Dynamixel TTL, J8 Dynamixel TTL, Q2 IPD068P03L3GATMA1, Q3 T2N7002AK, U7 SN74LV1T34, U8 SN74LVC2G241

Commit message: Fix PCBs.
Parts:
- added R2: 10k, Resistor_SMD:R_0805_2012Metric, symbol Device:R
Connections:
- net +5V: now also R2.1
- net at U7.2 (A), U8.6 (1Y): now also R2.2
Changed lines of the file:
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@@
   (junction (at 90.17 49.53) (diameter 0) (color 0 0 0 0)
   )
+  (junction (at 227.33 38.1) (diameter 0) (color 0 0 0 0)
+  )
   (junction (at 214.63 146.05) (diameter 0) (color 0 0 0 0)
   )
@@
     (stroke (width 0) (type default) (color 0 0 0 0))
   )
+  (wire (pts (xy 227.33 38.1) (xy 227.33 36.83))
+    (stroke (width 0) (type default) (color 0 0 0 0))
+  )
   (wire (pts (xy 213.36 133.35) (xy 215.9 133.35))
     (stroke (width 0) (type default) (color 0 0 0 0))
@@
   )
   (wire (pts (xy 186.69 60.96) (xy 184.15 60.96))
+    (stroke (width 0) (type default) (color 0 0 0 0))
+  )
+  (wire (pts (xy 227.33 26.67) (xy 227.33 29.21))
     (stroke (width 0) (type default) (color 0 0 0 0))
   )
@@
     (pin "2")
   )
+  (symbol (lib_id "power:+5V") (at 227.33 26.67 0) (unit 1)
+    (in_bom yes) (on_board yes) (fields_autoplaced)
+    (property "Reference" "#PWR0119" (id 0) (at 227.33 30.48 0)
+      (effects (font (size 1.27 1.27)) hide)
+    )
+    (property "Value" "+5V" (id 1) (at 227.33 21.59 0))
+    (property "Footprint" "" (id 2) (at 227.33 26.67 0)
+      (effects (font (size 1.27 1.27)) hide)
+    )
+    (property "Datasheet" "" (id 3) (at 227.33 26.67 0)
+      (effects (font (size 1.27 1.27)) hide)
+    )
+    (pin "1")
+  )
   (symbol (lib_id "Connector:Conn_01x03_Male") (at 177.8 107.95 0) (mirror x) (unit 1)
     (in_bom yes) (on_board yes) (fields_autoplaced)
@@
       (effects (font (size 1.27 1.27)) hide)
     )
+    (pin "1")
+    (pin "2")
+  )
+  (symbol (lib_id "Device:R") (at 227.33 33.02 0) (unit 1)
+    (in_bom yes) (on_board yes) (fields_autoplaced)
+    (property "Reference" "R2" (id 0) (at 229.87 31.7499 0)
+      (effects (font (size 1.27 1.27)) (justify left))
+    )
+    (property "Value" "10k" (id 1) (at 229.87 34.2899 0)
+      (effects (font (size 1.27 1.27)) (justify left))
+    )
+    (property "Footprint" "Resistor_SMD:R_0805_2012Metric" (id 2) (at 225.552 33.02 90)
+      (effects (font (size 1.27 1.27)) hide)
+    )
+    (property "Datasheet" "~" (id 3) (at 227.33 33.02 0)
+      (effects (font (size 1.27 1.27)) hide)
+    )
