File: PCB/psu_control/psu_control.kicad_pcb (KiCad board)
At the start: 4 copper layers, 100 x 70 mm, 113 parts, among them J1 Vin (10-25V), J10 Other 1 I2C, J11 Light Sensor Front, J12 Light Sensor Left, J13 Light Sensor Back, J14 Light Sensor Right, J15 RRC-PMM240, J16 RS232, J2 Vout (10-25V), J3 Vout (5V), J4 Vout (10-25V), J6 LED Strip, J7 Amplifier 2 I2C, J8 Amplifier 1 I2C, J9 Amplifier 2 I2C, M1 Fan, M2 Fan, Q1 SSM3J372R, Q2 IPD068P03L3GATMA1, Q3 T2N7002AK, Q4 AO4818B, SW1 Non-Momentary DPST, SW2 BUTTON, SW3 BUTTON, SW4 BUTTON, SW5 BUTTON, SW6 BUTTON, U1 LM810M3-4.63, U2 Teensy_LC, U3 INA220, U4 K7805-3AR3, U5 74HC14, U6 SN74LV1T34, U7 MAX3221E, U8 74LVC2G34

Commit message: PCB revision
Routing:
- net Net-(J15-Pad4): track 18.9 -> 13.7 mm
- net GND: track 91.5 -> 94.3 mm, vias 29 -> 31
- net Net-(C20-Pad1): track 2.75 -> 2.19 mm
Other:
- board text added: "RS232 TX RX G"
- board text added: "SDA SCL G"
- board text removed: "G SCL SDA"
- board text removed: "RS232 G RX TX"
Changed lines of the file:
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@@
     (property "Sheetname" "RS232")
     (attr smd)
-    (fp_text reference "U7" (at -0.55 3.5 90) (layer "F.SilkS")
+    (fp_text reference "U7" (at 0 -3.55 90) (layer "F.SilkS")
       (effects (font (size 1 1) (thickness 0.15)))
     )
@@
     (effects (font (size 1 1) (thickness 0.15)))
   )
-  (gr_text "RS232\nG RX TX" (at 105 59.25) (layer "F.SilkS")
+  (gr_text "RS232\nTX RX G" (at 105 59) (layer "F.SilkS")
     (effects (font (size 1 1) (thickness 0.15)) (justify left))
   )
@@
     (effects (font (size 1 1) (thickness 0.15)))
   )
-  (gr_text "G SCL SDA" (at 90.5 72 90) (layer "F.SilkS")
+  (gr_text "SDA SCL G" (at 90.5 72.25 90) (layer "F.SilkS")
     (effects (font (size 1 1) (thickness 0.15)))
   )
@@
   (segment (start 42.6 68) (end 41.5 68) (width 0.254) (layer "F.Cu") (net 2))
   (segment (start 55.05 44.5) (end 55.05 43.05) (width 0.254) (layer "F.Cu") (net 2))
+  (segment (start 107 46.55) (end 107 45.25) (width 0.508) (layer "F.Cu") (net 2))
   (segment (start 40 52.1) (end 41.4 52.1) (width 0.254) (layer "F.Cu") (net 2))
   (segment (start 110.25 58.6) (end 110.6 58.25) (width 0.381) (layer "F.Cu") (net 2))
@@
   (segment (start 111.425 56.1125) (end 111.425 55.331328) (width 0.381) (layer "F.Cu") (net 2))
   (segment (start 111.5 57.5) (end 111.5 58) (width 0.381) (layer "F.Cu") (net 2))
+  (segment (start 113.2 48.25) (end 113.2 48.394) (width 0.508) (layer "F.Cu") (net 2))
   (segment (start 105.4 28.9) (end 105.5 29) (width 1.27) (layer "F.Cu") (net 2))
   (segment (start 102.9 35) (end 104 35) (width 0.508) (layer "F.Cu") (net 2))
@@
   (segment (start 110.75 53.75) (end 111.25 53.75) (width 0.381) (layer "F.Cu") (net 2))
   (segment (start 110 59.5) (end 110.5 59.5) (width 0.381) (layer "F.Cu") (net 2))
+  (segment (start 113.2 49.2) (end 113.5 49.5) (width 0.508) (layer "F.Cu") (net 2))
+  (segment (start 113.2 48.25) (end 113.2 49.2) (width 0.508) (layer "F.Cu") (net 2))
   (segment (start 103.8625 39.6375) (end 104 39.5) (width 0.254) (layer "F.Cu") (net 2))
   (segment (start 111.5 58.5) (end 111 58) (width 0.381) (layer "F.Cu") (net 2))
@@
   (via (at 46.5 74) (size 0.6858) (drill 0.3302) (layers "F.Cu" "B.Cu") (net 2))
   (via (at 104 35) (size 0.889) (drill 0.381) (layers "F.Cu" "B.Cu") (net 2))
+  (via (at 107 45.25) (size 0.889) (drill 0.381) (layers "F.Cu" "B.Cu") (net 2))
   (via (at 60 56) (size 0.6858) (drill 0.3302) (layers "F.Cu" "B.Cu") (net 2))
   (via (at 98.5 33) (size 0.6858) (drill 0.3302) (layers "F.Cu" "B.Cu") (net 2))
@@
   (via (at 104.25 18.5) (size 0.6858) (drill 0.3302) (layers "F.Cu" "B.Cu") (net 2))
   (via (at 41.5 68) (size 0.6858) (drill 0.3302) (layers "F.Cu" "B.Cu") (net 2))
+  (via (at 113.5 49.5) (size 0.889) (drill 0.381) (layers "F.Cu" "B.Cu") (net 2))
   (via (at 110 59.5) (size 0.6858) (drill 0.3302) (layers "F.Cu" "B.Cu") (net 2))
   (via (at 111.5 53.5) (size 0.6858) (drill 0.3302) (layers "F.Cu" "B.Cu") (net 2))
@@
   (segment (start 35.9125 33.5875) (end 35.4125 34.0875) (width 0.254) (layer "F.Cu") (net 6))
   (segment (start 35.4125 34.0875) (end 35.4125 35) (width 0.254) (layer "F.Cu") (net 6))
-  (segment (start 101 37.3125) (end 100.95 37.3625) (width 0.254) (layer "F.Cu") (net 7))
   (segment (start 106.9125 20) (end 106.9125 21.1625) (width 0.254) (layer "F.Cu") (net 7))
   (segment (start 77 28.5) (end 79 26.5) (width 1.27) (layer "F.Cu") (net 7))
@@
   (segment (start 108.198 48.489001) (end 108.535999 48.827) (width 0.254) (layer "F.Cu") (net 20))
   (segment (start 111.425 48.375) (end 111.3 48.25) (width 0.254) (layer "F.Cu") (net 21))
-  (segment (start 111.25 48.65) (end 110.85 48.25) (width 0.254) (layer "F.Cu") (net 21))
   (segment (start 111.425 50.3875) (end 111.425 48.375) (width 0.254) (layer "F.Cu") (net 21))
   (segment (start 107.2 48.45) (end 108.073 49.323) (width 0.254) (layer "F.Cu") (net 22))
@@
   (segment (start 34.25 28.25) (end 33.4125 29.0875) (width 0.254) (layer "F.Cu") (net 77))
   (segment (start 79.5 70.75) (end 79.5 70.95) (width 0.508) (layer "F.Cu") (net 78))
-  (segment (start 78.8 65.16) (end 78.8 69.55) (width 0.254) (layer "F.Cu") (net 78))
   (segment (start 85 69) (end 84.75 68.75) (width 0.508) (layer "F.Cu") (net 78))
-  (segment (start 81.88 68.62) (end 81.75 68.75) (width 0.254) (layer "F.Cu") (net 78))
-  (segment (start 79.5 70.25) (end 79.5 70.95) (width 0.254) (layer "F.Cu") (net 78))
   (segment (start 81.5 68.75) (end 79.5 70.75) (width 0.508) (layer "F.Cu") (net 78))
   (segment (start 84.75 68.75) (end 81.75 68.75) (width 0.508) (layer "F.Cu") (net 78))
@@
     (connect_pads yes (clearance 0.508))
     (min_thickness 0.254) (filled_areas_thickness no)
-    (fill (thermal_gap 0.508) (thermal_bridge_width 0.508))
+    (fill yes (thermal_gap 0.508) (thermal_bridge_width 0.508))
     (polygon
       (pts
@@
     (connect_pads yes (clearance 0.508))
     (min_thickness 0.254) (filled_areas_thickness no)
-    (fill (thermal_gap 0.508) (thermal_bridge_width 0.508))
+    (fill yes (thermal_gap 0.508) (thermal_bridge_width 0.508))
     (polygon
       (pts
@@
     (connect_pads yes (clearance 0.508))
     (min_thickness 0.254) (filled_areas_thickness no)
-    (fill (thermal_gap 0.508) (thermal_bridge_width 0.508))
+    (fill yes (thermal_gap 0.508) (thermal_bridge_width 0.508))
     (polygon
       (pts
@@
     (connect_pads yes (clearance 0.508))
     (min_thickness 0.254) (filled_areas_thickness no)
-    (fill (thermal_gap 0.508) (thermal_bridge_width 0.508))
+    (fill yes (thermal_gap 0.508) (thermal_bridge_width 0.508))
     (polygon
       (pts
@@
     (connect_pads yes (clearance 0.508))
     (min_thickness 0.254) (filled_areas_thickness no)
-    (fill (thermal_gap 0.508) (thermal_bridge_width 0.508))
+    (fill yes (thermal_gap 0.508) (thermal_bridge_width 0.508))
     (polygon
       (pts
@@
     (connect_pads yes (clearance 0.508))
     (min_thickness 0.254) (filled_areas_thickness no)
-    (fill (thermal_gap 0.508) (thermal_bridge_width 0.508))
+    (fill yes (thermal_gap 0.508) (thermal_bridge_width 0.508))
     (polygon
       (pts
@@
     (connect_pads yes (clearance 0.508))
     (min_thickness 0.254) (filled_areas_thickness no)
-    (fill (thermal_gap 0.508) (thermal_bridge_width 0.508))
+    (fill yes (thermal_gap 0.508) (thermal_bridge_width 0.508))
     (polygon
       (pts
@@
     (connect_pads yes (clearance 0.508))
     (min_thickness 0.254) (filled_areas_thickness no)
-    (fill (thermal_gap 0.508) (thermal_bridge_width 0.508))
+    (fill yes (thermal_gap 0.508) (thermal_bridge_width 0.508))
     (polygon
       (pts
@@
     (connect_pads yes (clearance 0.508))
     (min_thickness 0.254) (filled_areas_thickness no)
-    (fill (thermal_gap 0.508) (thermal_bridge_width 0.508))
+    (fill yes (thermal_gap 0.508) (thermal_bridge_width 0.508))
     (polygon
       (pts
@@
     (connect_pads yes (clearance 0.508))
     (min_thickness 0.254) (filled_areas_thickness no)
-    (fill (thermal_gap 0.508) (thermal_bridge_width 0.508))
+    (fill yes (thermal_gap 0.508) (thermal_bridge_width 0.508))
     (polygon
       (pts
@@
     (connect_pads yes (clearance 0.508))
     (min_thickness 0.254) (filled_areas_thickness no)
-    (fill (thermal_gap 0.508) (thermal_bridge_width 0.508))
+    (fill yes (thermal_gap 0.508) (thermal_bridge_width 0.508))
     (polygon
       (pts
@@
     (connect_pads yes (clearance 0.508))
     (min_thickness 0.254) (filled_areas_thickness no)
-    (fill (thermal_gap 0.508) (thermal_bridge_width 0.508))
+    (fill yes (thermal_gap 0.508) (thermal_bridge_width 0.508))
     (polygon
       (pts
@@
     (connect_pads yes (clearance 0.508))
     (min_thickness 0.254) (filled_areas_thickness no)
-    (fill (thermal_gap 0.508) (thermal_bridge_width 0.508))
+    (fill yes (thermal_gap 0.508) (thermal_bridge_width 0.508))
     (polygon
       (pts
@@
     (connect_pads yes (clearance 0.508))
     (min_thickness 0.254) (filled_areas_thickness no)
-    (fill (thermal_gap 0.508) (thermal_bridge_width 0.508))
+    (fill yes (thermal_gap 0.508) (thermal_bridge_width 0.508))
     (polygon
       (pts
@@
     (connect_pads yes (clearance 0.508))
     (min_thickness 0.254) (filled_areas_thickness no)
-    (fill (thermal_gap 0.508) (thermal_bridge_width 0.508))
+    (fill yes (thermal_gap 0.508) (thermal_bridge_width 0.508))
     (polygon
       (pts
@@
     (connect_pads yes (clearance 0.508))
     (min_thickness 0.254) (filled_areas_thickness no)
-    (fill (thermal_gap 0.508) (thermal_bridge_width 0.508))
+    (fill yes (thermal_gap 0.508) (thermal_bridge_width 0.508))
     (polygon
       (pts
