File: PCB/psu_control/psu_control.kicad_sch (KiCad schematic)
At the start: 7 parts

Commit message: psu_control v4 is completed
Parts:
- removed U?: Teensy_LC, symbol t-top:Teensy_LC
- added U2: Teensy_LC, t-top:Teensy_LC, symbol t-top:Teensy_LC
- Q1: renamed from Q?; footprint (none) -> Package_TO_SOT_SMD:SOT-23
- R1, R2: renamed from R?; footprint (none) -> Resistor_SMD:R_0805_2012Metric
- R3, R4: renamed from R?; value 1k -> 2.2k; footprint (none) -> Resistor_SMD:R_0805_2012Metric
- U1: renamed from U?; footprint (none) -> Package_TO_SOT_SMD:SOT-23
Connections:
- net +3.3V: now also U2.3V3_1 (3V3)
- net Actuators/BUZZER_PWM: now also U2.6 (6/CS1/PWM)
- net Actuators/FAN_PWM: now also U2.3 (3/PWM)
- net Actuators/LED_STRIP_DATA: now also U2.1 (1/TX1/MISO1)
- net Battery/BATTERY_SMBUS_SCL: now also U2.19 (19/A5/SCL0)
- net Battery/BATTERY_SMBUS_SDA: now also U2.18 (18/A4/SDA0)
- net Battery/BATTERY_STATUS: now also U2.20 (20/A6/SCK1/PWM)
- net Battery/CHARGER_STATUS: now also U2.21 (21/A7)
- net GENERAL_SCL: now also U2.22 (22/A8/SCL1/PWM)
- net GENERAL_SDA: now also U2.23 (23/A9/SDA1/PWM)
- net GND: now also U2.GND_1 (GND)
- net Sensors/EXTERNAL_TEMPERATURE: now also U2.15 (15/A1)
- net Sensors/LIGHT_SENSOR_FRONT: now also U2.16 (16/A2/PWM)
- net Sensors/LIGHT_SENSOR_LEFT: now also U2.17 (17/A3/PWM)
- net Sensors/ONBOARD_TEMPERATURE: now also U2.14 (14/A0)
- net at Q1.3 (D): now also U2.VIN
- new net BUTTON_OTHER: U2.13 (13/SCK0)
- new net BUTTON_START: U2.9 (9/RX2/PWM)
- new net BUTTON_STOP: U2.10 (10/TX2/CS0/PWM)
- new net BUTTON_VOLUME_DOWN: U2.11 (11/MOSI0)
- new net BUTTON_VOLUME_UP: U2.12 (12/MISO0)
- new net LIGHT_SENSOR_BACK: U2.25 (25/A11)
- new net LIGHT_SENSOR_RIGHT: U2.24 (24/A10)
- new net POWER_SWITCH: U2.4 (4/PWM)
- new net RS232/UART_RX: U2.7 (7/RX3)
- new net RS232/UART_TX: U2.8 (8/TX3)
- new net ~{POWER_OFF}: U2.2
- new net ~{RS232_INVALID}: U2.5
- no-connect marks 1 -> 3
Other:
- added sheet RS232 (rs232.kicad_sch)

Commit message: Fix issues. Add schematic files.
Changed lines of the file:
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@@
+    (stroke (width 0) (type default) (color 0 0 0 0))
+  )
+  (wire (pts (xy 99.06 81.28) (xy 100.33 81.28))
     (stroke (width 0) (type default) (color 0 0 0 0))
   )
@@
     (stroke (width 0) (type default) (color 0 0 0 0))
   )
+  (wire (pts (xy 99.06 86.36) (xy 100.33 86.36))
+    (stroke (width 0) (type default) (color 0 0 0 0))
+  )
+  (wire (pts (xy 99.06 88.9) (xy 100.33 88.9))
+    (stroke (width 0) (type default) (color 0 0 0 0))
+  )
   (wire (pts (xy 208.28 82.55) (xy 208.28 86.36))
     (stroke (width 0) (type default) (color 0 0 0 0))
@@
     (stroke (width 0) (type default) (color 0 0 0 0))
   )
-  (label "~{POWER_OFF}" (at 100.33 81.28 180)
+  (label "~{POWER_OFF}" (at 99.06 81.28 180)
     (effects (font (size 1.27 1.27)) (justify right bottom))
   )
@@
     (effects (font (size 1.27 1.27)) (justify right bottom))
   )
-  (label "~{RS232_INVALID}" (at 100.33 88.9 180)
+  (label "~{RS232_INVALID}" (at 99.06 88.9 180)
     (effects (font (size 1.27 1.27)) (justify right bottom))
   )
@@
     (effects (font (size 1.27 1.27)) (justify right bottom))
   )
-  (label "POWER_SWITCH" (at 100.33 86.36 180)
+  (label "POWER_SWITCH" (at 99.06 86.36 180)
     (effects (font (size 1.27 1.27)) (justify right bottom))
   )

Commit message: Fix PCBs.
Connections:
- net BUTTON_START: now also U2.11 (11/MOSI0); no longer U2.9 (9/RX2/PWM)
- net BUTTON_VOLUME_DOWN: now also U2.4 (4/PWM); no longer U2.11 (11/MOSI0)
- net BUTTON_VOLUME_UP: now also U2.9 (9/RX2/PWM); no longer U2.12 (12/MISO0)
- net POWER_SWITCH: now also U2.12 (12/MISO0); no longer U2.4 (4/PWM)
