File: PCB/buck_boost/buck_boost.kicad_pcb (KiCad board)
At the start: 4 copper layers, 80 x 70 mm, 60 parts, among them J1 VIN 10-24V, J2 VOUT, J3 VOUT, J4 VOUT, J5 VOUT, Q1 TK1R4S04PB, Q2 TK1R4S04PB, Q3 TK1R4S04PB, Q4 TK1R4S04PB, Q5 TK1R4S04PB, U1 LTC4359-MS8, U2 LT8392

Commit message: t top v4 (#76)
* Add the CAD files of the base.

* Add Jetson AGX Orin

* Move torso magnets to the outer diameter.

* Rename support to bracket

* Add stewart bottom

* Fix torso bottom holder

* Add the head onto the stewart platform. Add the stewart platform onto the robots.

* Add magnets on the head

* Add stewart springs.

* Apply comments

* Fix CAD. Add STL.

* Rename CAD_v4 to CAD

* Update buck_boost to kicad 6

* Add first draft of psu_control

* psu_control v4 is completed

* Update psu_control

* Add dynamixel_control PCB

* Add dynamixel control to CAD.

* Fix issues. Add schematic files.

* Fix pdf

* Add the serial MCU communucation protocol.

* Fix SERIAL_MCU.md

* Fix SERIAL_MCU.md

* Update psu_control

* Add acknowledgment payload to SERIAL_MCU.md.

* Add preamble and volume maximum to SERIAL_MCU.md

* Update SERIAL_MCU.md. Add the electrical block diagram.

* PCB revision

* Remove old psu_control gerber files.

* Remove the old part lib file

* Create gerber files for psu_control and dynamixel_control.

* Add SERVICE_ROS.md

* Add the beginning of the serial communication code.

* Update submodules.

* Add message classes.

* building common message library, daemon incomplete

* Opening serial port

* Skeleton for system tray

* Some menu working

* Connecting to daemon, WIP

* Connecting to daemon, WIP

* Add almost all PSU control code.

* Fix PushButton::read()

* Add output resistor for the led strip (data).

* Update gerbers

* Fix T-Connector

* Add Debug UART connector to dynamixel_control.

* Update schematics.

* Change MAX3221E by SN65C3221E.

* Add SerialCommunicationManager

* Fix missing include and common files

* Fix PCBs.

* Update psu control. Add missing CAD files.

* Add a PI filter to buck_boost. Fix ringing for other PI filters.

* Refs #47 first integration with Qt. Not processing messages, why?

* Refs #47 first i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
Parts:
- added L2: 1µH (PA4987.102HLT), t-top:PA4987.XXXHL, F.Cu at (86.5, 44.5)
- D2, D3: value SMD24PL-TP -> SS2040LL
- L1: value 15µF -> 15µH (PQ2617BHA-150K)
- moved C11 7.50 mm to (89.5, 55.5)
- moved RV1 6.79 mm to (88.0, 65.3)
- moved C4 5.44 mm to (86.5, 68.8), turned to -90 degrees
- moved Q1 2.73 mm to (88.2, 76.2)
- moved U1 1.97 mm to (81.6, 68.8)
- moved JP1 1.75 mm to (86.0, 81.2)
- moved C25 1.00 mm to (89.5, 33.5)
- moved C19 0.75 mm to (72.5, 76.2)
Connections:
- net /~PGOOD renamed /~{PGOOD}
- C25 pad 1: Net-(C11-Pad1) -> Net-(C25-Pad1)
- J2 pad 2: Net-(C11-Pad1) -> Net-(C25-Pad1)
- J3 pad 2: Net-(C11-Pad1) -> Net-(C25-Pad1)
- J4 pad 2: Net-(C11-Pad1) -> Net-(C25-Pad1)
- J5 pad 2: Net-(C11-Pad1) -> Net-(C25-Pad1)
- RV2 pad 3: Net-(RV2-Pad3) -> unconnected-(RV2-Pad3)
- U1 pad 3: Net-(U1-Pad3) -> unconnected-(U1-Pad3)
- U1 pad 7: Net-(U1-Pad7) -> unconnected-(U1-Pad7)
- U2 pad 16: Net-(U2-Pad16) -> unconnected-(U2-Pad16)
Routing:
- net Net-(Q1-Pad1): track 7.69 -> 9.59 mm
- net GNDPWR: track 59.7 -> 61.3 mm, vias 52 -> 51
- net /REG_OUT: track 56.3 -> 57.8 mm, vias 3 -> 2
- net Net-(C11-Pad1): track 1.36 -> 2.77 mm
- net +5V: track 47.5 -> 46.1 mm
- net Net-(C18-Pad1): track 47.6 -> 48.8 mm
- added copper zone on F.Cu, net Net-(C25-Pad1)
Other:
- net class Default removed
